File: ADSR.kicad_pcb (KiCad board)
At the start: 2 copper layers, 9.9 x 110.1 mm, 44 parts, among them J1 Gate, J2 Out, J3 EuroPower, Q1 MMBT3904, Q2 MMBT3904, Q3 MMBT3904, Q4 MMBT3904, U1 NE555, U2 LM358

Commit message: Make width 10mm, use SOD-123 package diodes
Other:
- board size 9.9 x 110.1 mm -> 10 x 110.1 mm
- net class Default removed
